Commit message: Revert "Add PI macro"
This reverts commit c78ad0cfbff4e22e27ff9f73b5c7331a03dcb6a1.

File: xarm_description/urdf/xarm7_robot_macro.xacro (robot description, xacro)
@@ -12,5 +12,4 @@
     geometry_mesh_tcp_xyz:='0 0 0'
     geometry_mesh_tcp_rpy:='0 0 0' ">
-    <xacro:property name="pi" value="3.1415" />
     <!-- xarm7 -->
     <xacro:include filename="$(find xarm_description)/urdf/xarm7.urdf.xacro" />

Commit message: Add PI macro

File: xarm_description/urdf/xarm7_robot_macro.xacro (robot description, xacro)
@@ -12,4 +12,5 @@
     geometry_mesh_tcp_xyz:='0 0 0'
     geometry_mesh_tcp_rpy:='0 0 0' ">
+    <xacro:property name="pi" value="3.1415" />
     <!-- xarm7 -->
     <xacro:include filename="$(find xarm_description)/urdf/xarm7.urdf.xacro" />
