Commit message: wip

File: xarm_description/urdf/xarm7.urdf.xacro (robot description, xacro)
@@ -43,7 +43,4 @@
     </inertial>
     <visual>
-      <origin
-        xyz="0 0 0"
-        rpy="0 0 0" />
       <geometry>
         <mesh
@@ -53,7 +50,4 @@
     </visual>
     <collision>
-      <origin
-        xyz="0 0 0"
-        rpy="0 0 0" />
       <geometry>
         <mesh
@@ -62,9 +56,8 @@
     </collision>
   </link>
-  <link
-    name="${prefix}link1">
-    <inertial>
-      <origin
-        xyz="-0.0042 0.0282 0.1032"
+  <link name="${prefix}link1">
+    <inertial>
+      <origin
+        xyz="-0.0042 0.0282 0.0088"
         rpy="0 0 0" />
       <mass
@@ -79,7 +72,4 @@
     </inertial>
     <visual>
-      <origin
-        xyz="0 0 0.112"
-        rpy="0 0 0" />
       <geometry>
         <mesh
@@ -89,7 +79,4 @@
     </visual>
     <collision>
-      <origin
-        xyz="0 0 0.112"
-        rpy="0 0 0" />
       <geometry>
         <mesh
@@ -102,5 +89,5 @@
     type="revolute">
     <origin
-      xyz="0 0 0.155"
+      xyz="0 0 0.267"
       rpy="0 0 0" />
     <parent
@@ -123,5 +110,5 @@
     <inertial>
       <origin
-        xyz="0 -0.1285 -0.0487"
+        xyz="0 -0.1285 0.0267"
         rpy="0 0 0" />
       <mass
@@ -136,7 +123,4 @@
     </inertial>
     <visual>
-      <origin
-        xyz="0 0 -0.075"
-        rpy="0 0 0" />
       <geometry>
         <mesh
@@ -146,7 +130,4 @@
     </visual>
     <collision>
-      <origin
-        xyz="0 0 -0.075"
-        rpy="0 0 0" />
       <geometry>
         <mesh
@@ -159,5 +140,5 @@
     type="revolute">
     <origin
-      xyz="0 0.075 0.112"
+      xyz="0 0 0"
       rpy="-1.5708 0 0" />
     <parent
@@ -216,5 +197,5 @@
     type="revolute">
     <origin
-      xyz="0 -0.192 -0.075"
+      xyz="0 -0.192 0"
       rpy="1.5708 0 0" />
     <parent

Commit message: wip

File: xarm_description/urdf/xarm7.urdf.xacro (robot description, xacro)
@@ -161,5 +161,5 @@
     <inertial>
       <origin
-        xyz="0.0422 -0.0233 0.0913"
+        xyz="0.0422 -0.0233 -0.0097"
         rpy="0 0 0" />
       <mass
@@ -174,7 +174,4 @@
     </inertial>
     <visual>
-      <origin
-        xyz="0 0 0.101"
-        rpy="0 0 0" />
       <geometry>
         <mesh
@@ -184,7 +181,4 @@
     </visual>
     <collision>
-      <origin
-        xyz="0 0 0.101"
-        rpy="0 0 0" />
       <geometry>
         <mesh
@@ -197,5 +191,5 @@
     type="revolute">
     <origin
-      xyz="0 -0.192 0"
+      xyz="0 -0.293 0"
       rpy="1.5708 0 0" />
     <parent
@@ -254,5 +248,5 @@
     type="revolute">
     <origin
-      xyz="0.0525 -0.067 0.101"
+      xyz="0.0525 -0.067 0"
       rpy="1.5708 0 0" />
     <parent

Commit message: wip

File: xarm_description/urdf/xarm7.urdf.xacro (robot description, xacro)
@@ -59,5 +59,5 @@
     <inertial>
       <origin
-        xyz="-0.0042 0.0282 0.0088"
+        xyz="-0.0042 0.0282 -0.0088"
         rpy="0 0 0" />
       <mass
@@ -212,5 +212,5 @@
     <inertial>
       <origin
-        xyz="0.0671 -0.1073 -0.0425"
+        xyz="0.0671 -0.1073 0.0245"
         rpy="0 0 0" />
       <mass
@@ -225,7 +225,4 @@
     </inertial>
     <visual>
-      <origin
-        xyz="0 0 -0.067"
-        rpy="0 0 0" />
       <geometry>
         <mesh
@@ -235,7 +232,4 @@
     </visual>
     <collision>
-      <origin
-        xyz="0 0 -0.067"
-        rpy="0 0 0" />
       <geometry>
         <mesh
@@ -248,5 +242,5 @@
     type="revolute">
     <origin
-      xyz="0.0525 -0.067 0"
+      xyz="0.0525 0 0"
       rpy="1.5708 0 0" />
     <parent
@@ -305,5 +299,5 @@
     type="revolute">
     <origin
-      xyz="0.0775 -0.169 -0.067"
+      xyz="0.0775 -0.169 0"
       rpy="1.5708 0 0" />
     <parent

Commit message: wip

File: xarm_description/urdf/xarm7.urdf.xacro (robot description, xacro)
@@ -263,5 +263,5 @@
     <inertial>
       <origin
-        xyz="-0.0002 0.0367 0.0929"
+        xyz="-0.0002 0.0367 -0.0801"
         rpy="0 0 0" />
       <mass
@@ -276,7 +276,4 @@
     </inertial>
     <visual>
-      <origin
-        xyz="0 0 0.173"
-        rpy="0 0 0" />
       <geometry>
         <mesh
@@ -286,7 +283,4 @@
     </visual>
     <collision>
-      <origin
-        xyz="0 0 0.173"
-        rpy="0 0 0" />
       <geometry>
         <mesh
@@ -299,5 +293,5 @@
     type="revolute">
     <origin
-      xyz="0.0775 -0.169 0"
+      xyz="0.0775 -0.342 0"
       rpy="1.5708 0 0" />
     <parent
@@ -356,5 +350,5 @@
     type="revolute">
     <origin
-      xyz="0 0 0.173"
+      xyz="0 0 0"
       rpy="1.5708 0 0" />
     <parent

Commit message: finish

File: xarm_description/urdf/xarm7.urdf.xacro (robot description, xacro)
@@ -327,7 +327,4 @@
     </inertial>
     <visual>
-      <origin
-        xyz="0 0 0"
-        rpy="0 0 0" />
       <geometry>
         <mesh
@@ -337,7 +334,4 @@
     </visual>
     <collision>
-      <origin
-        xyz="0 0 0"
-        rpy="0 0 0" />
       <geometry>
         <mesh
@@ -371,5 +365,5 @@
     <inertial>
       <origin
-        xyz="0 -0.0046 0.0153"
+        xyz="0 -0.0046 -0.0127"
         rpy="0 0 0" />
       <mass
@@ -384,7 +378,4 @@
     </inertial>
     <visual>
-      <origin
-        xyz="0 0 0.028"
-        rpy="0 0 0" />
       <geometry>
         <mesh
@@ -394,7 +385,4 @@
     </visual>
     <collision>
-      <origin
-        xyz="0 0 0.028"
-        rpy="0 0 0" />
       <geometry>
         <mesh
@@ -407,5 +395,5 @@
     type="revolute">
     <origin
-      xyz="0.076 0.069 0"
+      xyz="0.076 0.097 0"
       rpy="-1.5708 0 0" />
     <parent
@@ -454,5 +442,5 @@
     type="fixed">
     <origin
-      xyz="0 0 0.028"
+      xyz="0 0 0"
       rpy="0 0 0" />
     <parent
