Commit message: collide without contact

File: xarm_description/urdf/xarm7.gazebo.xacro (robot description, xacro)
@@ -4,25 +4,81 @@
     <gazebo reference="${prefix}link_base">
       <selfCollide>false</selfCollide>
+      <collision>
+        <surface>
+          <contact>
+            <collide_without_contact>true</collide_without_contact>
+          </contact>
+        </surface>
+      </collision>
     </gazebo>
     <gazebo reference="${prefix}link1">
       <selfCollide>false</selfCollide>
+      <collision>
+        <surface>
+          <contact>
+            <collide_without_contact>true</collide_without_contact>
+          </contact>
+        </surface>
+      </collision>
     </gazebo>
     <gazebo reference="${prefix}link2">
       <selfCollide>false</selfCollide>
+      <collision>
+        <surface>
+          <contact>
+            <collide_without_contact>true</collide_without_contact>
+          </contact>
+        </surface>
+      </collision>
     </gazebo>
     <gazebo reference="${prefix}link3">
       <selfCollide>false</selfCollide>
+      <collision>
+        <surface>
+          <contact>
+            <collide_without_contact>true</collide_without_contact>
+          </contact>
+        </surface>
+      </collision>
     </gazebo>
     <gazebo reference="${prefix}link4">
       <selfCollide>false</selfCollide>
+      <collision>
+        <surface>
+          <contact>
+            <collide_without_contact>true</collide_without_contact>
+          </contact>
+        </surface>
+      </collision>
     </gazebo>
     <gazebo reference="${prefix}link5">
       <selfCollide>false</selfCollide>
+      <collision>
+        <surface>
+          <contact>
+            <collide_without_contact>true</collide_without_contact>
+          </contact>
+        </surface>
+      </collision>
     </gazebo>
     <gazebo reference="${prefix}link6">
       <selfCollide>false</selfCollide>
+      <collision>
+        <surface>
+          <contact>
+            <collide_without_contact>true</collide_without_contact>
+          </contact>
+        </surface>
+      </collision>
     </gazebo>
     <gazebo reference="${prefix}link7">
       <selfCollide>false</selfCollide>
+      <collision>
+        <surface>
+          <contact>
+            <collide_without_contact>true</collide_without_contact>
+          </contact>
+        </surface>
+      </collision>
     </gazebo>
     <gazebo reference="${prefix}joint1">

File: xarm_gripper/urdf/xarm_gripper.gazebo.xacro (robot description, xacro)
@@ -49,7 +49,21 @@
     <gazebo reference="${prefix}xarm_gripper_base_link">
       <selfCollide>false</selfCollide>
+      <collision>
+        <surface>
+          <contact>
+            <collide_without_contact>true</collide_without_contact>
+          </contact>
+        </surface>
+      </collision>
     </gazebo>
     <gazebo reference="${prefix}left_outer_knuckle">
       <selfCollide>false</selfCollide>
+      <collision>
+        <surface>
+          <contact>
+            <collide_without_contact>true</collide_without_contact>
+          </contact>
+        </surface>
+      </collision>
     </gazebo>
     <gazebo reference="${prefix}left_finger">
@@ -63,10 +77,31 @@
       <selfCollide>false</selfCollide>
       <dampingFactor>0</dampingFactor>
+      <collision>
+        <surface>
+          <contact>
+            <collide_without_contact>true</collide_without_contact>
+          </contact>
+        </surface>
+      </collision>
     </gazebo>
     <gazebo reference="${prefix}left_inner_knuckle">
       <selfCollide>false</selfCollide>
+      <collision>
+        <surface>
+          <contact>
+            <collide_without_contact>true</collide_without_contact>
+          </contact>
+        </surface>
+      </collision>
     </gazebo>
     <gazebo reference="${prefix}right_outer_knuckle">
       <selfCollide>false</selfCollide>
+      <collision>
+        <surface>
+          <contact>
+            <collide_without_contact>true</collide_without_contact>
+          </contact>
+        </surface>
+      </collision>
     </gazebo>
     <gazebo reference="${prefix}right_finger">
@@ -80,7 +115,21 @@
       <selfCollide>false</selfCollide>
       <dampingFactor>0</dampingFactor>
+      <collision>
+        <surface>
+          <contact>
+            <collide_without_contact>true</collide_without_contact>
+          </contact>
+        </surface>
+      </collision>
     </gazebo>
     <gazebo reference="${prefix}right_inner_knuckle">
       <selfCollide>false</selfCollide>
+      <collision>
+        <surface>
+          <contact>
+            <collide_without_contact>true</collide_without_contact>
+          </contact>
+        </surface>
+      </collision>
     </gazebo>
     <gazebo reference="${prefix}drive_joint">

Commit message: added option

File: xarm_description/urdf/xarm7.gazebo.xacro (robot description, xacro)
@@ -1,84 +1,100 @@
 <?xml version="1.0"?>
 <robot xmlns:xacro="http://ros.org/wiki/xacro">
-  <xacro:macro name="xarm7_gazebo" params="prefix">
+  <xacro:macro name="xarm7_gazebo" params="prefix collide_without_contact:='false'">
     <gazebo reference="${prefix}link_base">
       <selfCollide>false</selfCollide>
-      <collision>
-        <surface>
-          <contact>
-            <collide_without_contact>true</collide_without_contact>
-          </contact>
-        </surface>
-      </collision>
+      <xacro:if value="${collide_without_contact}">
+        <collision>
+          <surface>
+            <contact>
+              <collide_without_contact>true</collide_without_contact>
+            </contact>
+          </surface>
+        </collision>
+      </xacro:if>
     </gazebo>
     <gazebo reference="${prefix}link1">
       <selfCollide>false</selfCollide>
-      <collision>
-        <surface>
-          <contact>
-            <collide_without_contact>true</collide_without_contact>
-          </contact>
-        </surface>
-      </collision>
+      <xacro:if value="${collide_without_contact}">
+        <collision>
+          <surface>
+            <contact>
+              <collide_without_contact>true</collide_without_contact>
+            </contact>
+          </surface>
+        </collision>
+      </xacro:if>
     </gazebo>
     <gazebo reference="${prefix}link2">
       <selfCollide>false</selfCollide>
-      <collision>
-        <surface>
-          <contact>
-            <collide_without_contact>true</collide_without_contact>
-          </contact>
-        </surface>
-      </collision>
+      <xacro:if value="${collide_without_contact}">
+        <collision>
+          <surface>
+            <contact>
+              <collide_without_contact>true</collide_without_contact>
+            </contact>
+          </surface>
+        </collision>
+      </xacro:if>
     </gazebo>
     <gazebo reference="${prefix}link3">
       <selfCollide>false</selfCollide>
-      <collision>
-        <surface>
-          <contact>
-            <collide_without_contact>true</collide_without_contact>
-          </contact>
-        </surface>
-      </collision>
+      <xacro:if value="${collide_without_contact}">
+        <collision>
+          <surface>
+            <contact>
+              <collide_without_contact>true</collide_without_contact>
+            </contact>
+          </surface>
+        </collision>
+      </xacro:if>
     </gazebo>
     <gazebo reference="${prefix}link4">
       <selfCollide>false</selfCollide>
-      <collision>
-        <surface>
-          <contact>
-            <collide_without_contact>true</collide_without_contact>
-          </contact>
-        </surface>
-      </collision>
+      <xacro:if value="${collide_without_contact}">
+        <collision>
+          <surface>
+            <contact>
+              <collide_without_contact>true</collide_without_contact>
+            </contact>
+          </surface>
+        </collision>
+      </xacro:if>
     </gazebo>
     <gazebo reference="${prefix}link5">
       <selfCollide>false</selfCollide>
-      <collision>
-        <surface>
-          <contact>
-            <collide_without_contact>true</collide_without_contact>
-          </contact>
-        </surface>
-      </collision>
+      <xacro:if value="${collide_without_contact}">
+        <collision>
+          <surface>
+            <contact>
+              <collide_without_contact>true</collide_without_contact>
+            </contact>
+          </surface>
+        </collision>
+      </xacro:if>
     </gazebo>
     <gazebo reference="${prefix}link6">
       <selfCollide>false</selfCollide>
-      <collision>
-        <surface>
-          <contact>
-            <collide_without_contact>true</collide_without_contact>
-          </contact>
-        </surface>
-      </collision>
+      <xacro:if value="${collide_without_contact}">
+        <collision>
+          <surface>
+            <contact>
+              <collide_without_contact>true</collide_without_contact>
+            </contact>
+          </surface>
+        </collision>
+      </xacro:if>
     </gazebo>
     <gazebo reference="${prefix}link7">
       <selfCollide>false</selfCollide>
-      <collision>
-        <surface>
-          <contact>
-            <collide_without_contact>true</collide_without_contact>
-          </contact>
-        </surface>
-      </collision>
+      <xacro:if value="${collide_without_contact}">
+        <collision>
+          <surface>
+            <contact>
+              <collide_without_contact>true</collide_without_contact>
+            </contact>
+          </surface>
+        </collision>
+      </xacro:if>
     </gazebo>
     <gazebo reference="${prefix}joint1">

File: xarm_description/urdf/xarm7_robot_macro.xacro (robot description, xacro)
@@ -11,5 +11,7 @@
     geometry_mesh_origin_rpy:='0 0 0'
     geometry_mesh_tcp_xyz:='0 0 0'
-    geometry_mesh_tcp_rpy:='0 0 0' ">
+    geometry_mesh_tcp_rpy:='0 0 0'
+    collide_without_contact:='false'
+    ">
     <!-- xarm7 -->
     <xacro:include filename="$(find xarm_description)/urdf/xarm7.urdf.xacro" />
@@ -45,5 +47,5 @@
     </xacro:unless>
     <xacro:xarm7_transmission prefix="${prefix}" hard_interface="$(eval 'EffortJointInterface' if ${effort_control} else 'VelocityJointInterface' if ${velocity_control} else 'PositionJointInterface')" />
-    <xacro:xarm7_gazebo prefix="${prefix}" />
+    <xacro:xarm7_gazebo prefix="${prefix}" collide_without_contact="${collide_without_contact}" />
     <xacro:if value="${add_other_geometry}">
       <xacro:include filename="$(find xarm_description)/urdf/other_geometry.urdf.xacro" />

File: xarm_gripper/urdf/xarm_gripper.gazebo.xacro (robot description, xacro)
@@ -46,24 +46,28 @@
     </gazebo>
   </xacro:macro>
-  <xacro:macro name="xarm_gripper_gazebo" params="prefix">
+  <xacro:macro name="xarm_gripper_gazebo" params="prefix collide_without_contact:='false'">
     <gazebo reference="${prefix}xarm_gripper_base_link">
       <selfCollide>false</selfCollide>
-      <collision>
-        <surface>
-          <contact>
-            <collide_without_contact>true</collide_without_contact>
-          </contact>
-        </surface>
-      </collision>
+      <xacro:if value="${collide_without_contact}">
+        <collision>
+          <surface>
+            <contact>
+              <collide_without_contact>true</collide_without_contact>
+            </contact>
+          </surface>
+        </collision>
+      </xacro:if>
     </gazebo>
     <gazebo reference="${prefix}left_outer_knuckle">
       <selfCollide>false</selfCollide>
-      <collision>
-        <surface>
-          <contact>
-            <collide_without_contact>true</collide_without_contact>
-          </contact>
-        </surface>
-      </collision>
+      <xacro:if value="${collide_without_contact}">
+        <collision>
+          <surface>
+            <contact>
+              <collide_without_contact>true</collide_without_contact>
+            </contact>
+          </surface>
+        </collision>
+      </xacro:if>
     </gazebo>
     <gazebo reference="${prefix}left_finger">
@@ -77,31 +81,37 @@
       <selfCollide>false</selfCollide>
       <dampingFactor>0</dampingFactor>
-      <collision>
-        <surface>
-          <contact>
-            <collide_without_contact>true</collide_without_contact>
-          </contact>
-        </surface>
-      </collision>
+      <xacro:if value="${collide_without_contact}">
+        <collision>
+          <surface>
+            <contact>
+              <collide_without_contact>true</collide_without_contact>
+            </contact>
+          </surface>
+        </collision>
+      </xacro:if>
     </gazebo>
     <gazebo reference="${prefix}left_inner_knuckle">
       <selfCollide>false</selfCollide>
-      <collision>
-        <surface>
-          <contact>
-            <collide_without_contact>true</collide_without_contact>
-          </contact>
-        </surface>
-      </collision>
+      <xacro:if value="${collide_without_contact}">
+        <collision>
+          <surface>
+            <contact>
+              <collide_without_contact>true</collide_without_contact>
+            </contact>
+          </surface>
+        </collision>
+      </xacro:if>
     </gazebo>
     <gazebo reference="${prefix}right_outer_knuckle">
       <selfCollide>false</selfCollide>
-      <collision>
-        <surface>
-          <contact>
-            <collide_without_contact>true</collide_without_contact>
-          </contact>
-        </surface>
-      </collision>
+      <xacro:if value="${collide_without_contact}">
+        <collision>
+          <surface>
+            <contact>
+              <collide_without_contact>true</collide_without_contact>
+            </contact>
+          </surface>
+        </collision>
+      </xacro:if>
     </gazebo>
     <gazebo reference="${prefix}right_finger">
@@ -115,21 +125,25 @@
       <selfCollide>false</selfCollide>
       <dampingFactor>0</dampingFactor>
-      <collision>
-        <surface>
-          <contact>
-            <collide_without_contact>true</collide_without_contact>
-          </contact>
-        </surface>
-      </collision>
+      <xacro:if value="${collide_without_contact}">
+        <collision>
+          <surface>
+            <contact>
+              <collide_without_contact>true</collide_without_contact>
+            </contact>
+          </surface>
+        </collision>
+      </xacro:if>
     </gazebo>
     <gazebo reference="${prefix}right_inner_knuckle">
       <selfCollide>false</selfCollide>
-      <collision>
-        <surface>
-          <contact>
-            <collide_without_contact>true</collide_without_contact>
-          </contact>
-        </surface>
-      </collision>
+      <xacro:if value="${collide_without_contact}">
+        <collision>
+          <surface>
+            <contact>
+              <collide_without_contact>true</collide_without_contact>
+            </contact>
+          </surface>
+        </collision>
+      </xacro:if>
     </gazebo>
     <gazebo reference="${prefix}drive_joint">

File: xarm_gripper/urdf/xarm_gripper_model.xacro (robot description, xacro)
@@ -8,10 +8,10 @@
   <xacro:include filename="$(find xarm_gripper)/urdf/xarm_gripper.transmission.xacro" />
   <xacro:include filename="$(find xarm_gripper)/urdf/xarm_gripper.gazebo.xacro" />
-  <xacro:macro name="load_gripper" params="prefix:='' attach_to:='' ns:='xarm' xyz:='0 0 0' rpy:='0 0 0' effort_control:='false' velocity_control:='false' robot_dof:=7 palm_link:='' loop_joints:='true'">
+  <xacro:macro name="load_gripper" params="prefix:='' attach_to:='' ns:='xarm' xyz:='0 0 0' rpy:='0 0 0' effort_control:='false' velocity_control:='false' robot_dof:=7 palm_link:='' loop_joints:='true' collide_without_contact:='false'">
     <!-- gazebo plugin -->
     <!-- <xacro:gazebo_ros_control_plugin namespace="${ns}"/> -->
     <xacro:xarm_gripper_urdf prefix="${prefix}" attach_to="${attach_to}" xyz="${xyz}" rpy="${rpy}" loop_joints="${loop_joints}" />
     <xacro:xarm_gripper_transmission prefix="${prefix}" hard_interface="$(eval 'EffortJointInterface' if ${effort_control} else 'VelocityJointInterface' if ${velocity_control} else 'PositionJointInterface')" />
-    <xacro:xarm_gripper_gazebo prefix="${prefix}" />
+    <xacro:xarm_gripper_gazebo prefix="${prefix}" collide_without_contact="${collide_without_contact}" />
     <xacro:if value="${palm_link == ''}">
       <xacro:xarm_gazebo_grasp_fix prefix="${prefix}" palm_link="${prefix}link${robot_dof}" />
