Commit message: added option to manual define palm link

File: xarm_gripper/urdf/xarm_gripper_model.xacro (robot description, xacro)
@@ -8,5 +8,5 @@
   <xacro:include filename="$(find xarm_gripper)/urdf/xarm_gripper.transmission.xacro" />
   <xacro:include filename="$(find xarm_gripper)/urdf/xarm_gripper.gazebo.xacro" />
-  <xacro:macro name="load_gripper" params="prefix:='' attach_to:='' ns:='xarm' xyz:='0 0 0' rpy:='0 0 0' effort_control:='false' velocity_control:='false' robot_dof:=7 ">
+  <xacro:macro name="load_gripper" params="prefix:='' attach_to:='' ns:='xarm' xyz:='0 0 0' rpy:='0 0 0' effort_control:='false' velocity_control:='false' robot_dof:=7 palm_link:=''">
     <!-- gazebo plugin -->
     <!-- <xacro:gazebo_ros_control_plugin namespace="${ns}"/> -->
@@ -14,5 +14,10 @@
     <xacro:xarm_gripper_transmission prefix="${prefix}" hard_interface="$(eval 'EffortJointInterface' if ${effort_control} else 'VelocityJointInterface' if ${velocity_control} else 'PositionJointInterface')" />
     <xacro:xarm_gripper_gazebo prefix="${prefix}" />
-    <xacro:xarm_gazebo_grasp_fix prefix="${prefix}" palm_link="${prefix}link${robot_dof}" />
+    <xacro:if value="${palm_link == ''}">
+      <xacro:xarm_gazebo_grasp_fix prefix="${prefix}" palm_link="${prefix}link${robot_dof}" />
+    </xacro:if>
+    <xacro:unless value="${palm_link == ''}">
+      <xacro:xarm_gazebo_grasp_fix prefix="${prefix}" palm_link="${palm_link}" />
+    </xacro:unless>
     <!-- mimic_joint_plugin has to be installed: -->
     <xacro:mimic_joint_plugin_gazebo name_prefix="${prefix}left_finger_joint"
