Commit message: Add gripper joint damping

File: xarm_gripper/urdf/xarm_gripper.gazebo.xacro (robot description, xacro)
@@ -84,4 +84,22 @@
       <selfCollide>false</selfCollide>
     </gazebo>
+    <gazebo reference="${prefix}drive_joint">
+      <implicitSpringDamper>1</implicitSpringDamper>
+    </gazebo>
+    <gazebo reference="${prefix}left_finger_joint">
+      <implicitSpringDamper>1</implicitSpringDamper>
+    </gazebo>
+    <gazebo reference="${prefix}left_inner_knuckle_joint">
+      <implicitSpringDamper>1</implicitSpringDamper>
+    </gazebo>
+    <gazebo reference="${prefix}right_outer_knuckle_joint">
+      <implicitSpringDamper>1</implicitSpringDamper>
+    </gazebo>
+    <gazebo reference="${prefix}right_finger_joint">
+      <implicitSpringDamper>1</implicitSpringDamper>
+    </gazebo>
+    <gazebo reference="${prefix}right_inner_knuckle_joint">
+      <implicitSpringDamper>1</implicitSpringDamper>
+    </gazebo>
   </xacro:macro>
 </robot>

File: xarm_gripper/urdf/xarm_gripper.urdf.xacro (robot description, xacro)
@@ -108,4 +108,7 @@
       effort="50"
       velocity="2" />
+    <dynamics
+      damping="1.0"
+      friction="0" />
   </joint>
   <link
@@ -171,4 +174,7 @@
       effort="50"
       velocity="2" />
+    <dynamics
+      damping="1.0"
+      friction="0" />
     <mimic joint="${prefix}drive_joint" multiplier="1" offset="0" />
   </joint>
@@ -227,4 +233,7 @@
       effort="50"
       velocity="2" />
+    <dynamics
+      damping="1.0"
+      friction="0" />
     <mimic joint="${prefix}drive_joint" multiplier="1" offset="0" />
   </joint>
@@ -283,4 +292,7 @@
       effort="50"
       velocity="2" />
+    <dynamics
+      damping="1.0"
+      friction="0" />
     <mimic joint="${prefix}drive_joint" multiplier="1" offset="0" />
   </joint>
@@ -347,4 +359,7 @@
       effort="50"
       velocity="2" />
+    <dynamics
+      damping="1.0"
+      friction="0" />
     <mimic joint="${prefix}drive_joint" multiplier="1" offset="0" />
   </joint>
@@ -403,4 +418,7 @@
       effort="50"
       velocity="2" />
+    <dynamics
+      damping="1.0"
+      friction="0" />
     <mimic joint="${prefix}drive_joint" multiplier="1" offset="0" />
   </joint>
