Commit message: Simplify gripper collision

File: xarm_gripper/urdf/xarm_gripper.urdf.xacro (robot description, xacro)
@@ -47,9 +47,8 @@
     <collision>
       <origin
-        xyz="0 0 0"
-        rpy="0 0 0" />
-      <geometry>
-        <mesh
-          filename="package://xarm_gripper/meshes/base_link_collision.STL" />
+        xyz="-0.0015 0 0.0515"
+        rpy="0 0 0" />
+      <geometry>
+        <box size="0.053 0.12 0.103"/>
       </geometry>
     </collision>
@@ -85,9 +84,8 @@
     <collision>
       <origin
-        xyz="0 0 0"
-        rpy="0 0 0" />
-      <geometry>
-        <mesh
-          filename="package://xarm_gripper/meshes/left_outer_knuckle.STL" />
+        xyz="0 0.015 0.02"
+        rpy="0.48 0 0" />
+      <geometry>
+        <box size="0.012 0.069 0.033"/>
       </geometry>
     </collision>
@@ -141,9 +139,16 @@
     <collision>
       <origin
-        xyz="0 0 0"
-        rpy="0 0 0" />
-      <geometry>
-        <mesh
-          filename="package://xarm_gripper/meshes/left_finger.STL" />
+        xyz="0 -0.019 0.04"
+        rpy="0 0 0" />
+      <geometry>
+        <box size="0.032 0.014 0.042"/>
+      </geometry>
+    </collision>
+    <collision>
+      <origin
+        xyz="0 -0.008 0.008"
+        rpy="0.8 0 0" />
+      <geometry>
+        <box size="0.016 0.012 0.036"/>
       </geometry>
     </collision>
@@ -198,9 +203,8 @@
     <collision>
       <origin
-        xyz="0 0 0"
-        rpy="0 0 0" />
-      <geometry>
-        <mesh
-          filename="package://xarm_gripper/meshes/left_inner_knuckle.STL" />
+        xyz="0 0.016 0.02"
+        rpy="-0.7 0 0" />
+      <geometry>
+        <box size="0.027 0.012 0.061"/>
       </geometry>
     </collision>
@@ -255,9 +259,8 @@
     <collision>
       <origin
-        xyz="0 0 0"
-        rpy="0 0 0" />
-      <geometry>
-        <mesh
-          filename="package://xarm_gripper/meshes/right_outer_knuckle.STL" />
+        xyz="0 -0.015 0.02"
+        rpy="-0.48 0 0" />
+      <geometry>
+        <box size="0.012 0.069 0.033"/>
       </geometry>
     </collision>
@@ -312,9 +315,16 @@
     <collision>
       <origin
-        xyz="0 0 0"
-        rpy="0 0 0" />
-      <geometry>
-        <mesh
-          filename="package://xarm_gripper/meshes/right_finger.STL" />
+        xyz="0 0.019 0.04"
+        rpy="0 0 0" />
+      <geometry>
+        <box size="0.032 0.014 0.042"/>
+      </geometry>
+    </collision>
+    <collision>
+      <origin
+        xyz="0 0.008 0.008"
+        rpy="-0.8 0 0" />
+      <geometry>
+        <box size="0.016 0.012 0.036"/>
       </geometry>
     </collision>
@@ -369,9 +379,8 @@
     <collision>
       <origin
-        xyz="0 0 0"
-        rpy="0 0 0" />
-      <geometry>
-        <mesh
-          filename="package://xarm_gripper/meshes/right_inner_knuckle.STL" />
+        xyz="0 -0.016 0.02"
+        rpy="0.7 0 0" />
+      <geometry>
+        <box size="0.027 0.012 0.061"/>
       </geometry>
     </collision>

Commit message: Add parallel link mechanism

File: xarm_gripper/urdf/xarm_gripper.urdf.xacro (robot description, xacro)
@@ -238,4 +238,25 @@
     <mimic joint="${prefix}drive_joint" multiplier="1" offset="0" />
   </joint>
+  <gazebo>
+    <joint name="${prefix}left_loop_joint" type="revolute">
+      <parent>${prefix}left_inner_knuckle</parent>
+      <child>${prefix}left_finger</child>
+      <pose>0 -0.015 0.015 0 0 0</pose>
+      <axis>
+        <xyz>1 0 0</xyz>
+        <use_parent_model_frame>true</use_parent_model_frame>
+      </axis>
+      <physics>
+        <ode>
+          <implicit_spring_damper>1</implicit_spring_damper>
+          <cfm_damping>0</cfm_damping>
+          <limit>
+            <cfm>1e-7</cfm>
+            <erp>0.8</erp>
+          </limit>
+        </ode>
+      </physics>
+    </joint>
+  </gazebo>
   <link
     name="${prefix}right_outer_knuckle">
@@ -423,4 +444,25 @@
     <mimic joint="${prefix}drive_joint" multiplier="1" offset="0" />
   </joint>
+  <gazebo>
+    <joint name="${prefix}right_loop_joint" type="revolute">
+      <parent>${prefix}right_inner_knuckle</parent>
+      <child>${prefix}right_finger</child>
+      <pose>0 0.015 0.015 0 0 0</pose>
+      <axis>
+        <xyz>1 0 0</xyz>
+        <use_parent_model_frame>true</use_parent_model_frame>
+      </axis>
+      <physics>
+        <ode>
+          <implicit_spring_damper>1</implicit_spring_damper>
+          <cfm_damping>0</cfm_damping>
+          <limit>
+            <cfm>1e-7</cfm>
+            <erp>0.8</erp>
+          </limit>
+        </ode>
+      </physics>
+    </joint>
+  </gazebo>
   <link name="${prefix}link_tcp" />
   <joint

File: xarm_gripper/urdf/xarm_gripper_model.xacro (robot description, xacro)
@@ -21,19 +21,19 @@
     </xacro:unless>
     <!-- mimic_joint_plugin has to be installed: -->
-    <xacro:mimic_joint_plugin_gazebo name_prefix="${prefix}left_finger_joint"
+<!--     <xacro:mimic_joint_plugin_gazebo name_prefix="${prefix}left_finger_joint"
       following_joint="${prefix}drive_joint" mimic_joint="${prefix}left_finger_joint"
-      has_pid="true" multiplier="1.0" max_effort="10.0" />
-    <xacro:mimic_joint_plugin_gazebo name_prefix="${prefix}left_inner_knuckle_joint"
+      has_pid="true" multiplier="1.0" max_effort="10.0" /> -->
+<!--     <xacro:mimic_joint_plugin_gazebo name_prefix="${prefix}left_inner_knuckle_joint"
       following_joint="${prefix}drive_joint" mimic_joint="${prefix}left_inner_knuckle_joint"
-      has_pid="true" multiplier="1.0" max_effort="10.0" />
+      has_pid="true" multiplier="1.0" max_effort="10.0" /> -->
     <xacro:mimic_joint_plugin_gazebo name_prefix="${prefix}right_outer_knuckle_joint"
       following_joint="${prefix}drive_joint" mimic_joint="${prefix}right_outer_knuckle_joint"
       has_pid="true" multiplier="1.0" max_effort="10.0" />
-    <xacro:mimic_joint_plugin_gazebo name_prefix="${prefix}right_finger_joint"
+<!--     <xacro:mimic_joint_plugin_gazebo name_prefix="${prefix}right_finger_joint"
       following_joint="${prefix}drive_joint" mimic_joint="${prefix}right_finger_joint"
-      has_pid="true" multiplier="1.0" max_effort="10.0" />
-    <xacro:mimic_joint_plugin_gazebo name_prefix="${prefix}right_inner_knuckle_joint"
+      has_pid="true" multiplier="1.0" max_effort="10.0" /> -->
+<!--     <xacro:mimic_joint_plugin_gazebo name_prefix="${prefix}right_inner_knuckle_joint"
       following_joint="${prefix}drive_joint" mimic_joint="${prefix}right_inner_knuckle_joint"
-      has_pid="true" multiplier="1.0" max_effort="10.0" />
+      has_pid="true" multiplier="1.0" max_effort="10.0" /> -->
   </xacro:macro>
 </robot>

Commit message: Add loop_joints option

File: xarm_gripper/urdf/xarm_gripper.urdf.xacro (robot description, xacro)
@@ -4,5 +4,5 @@
   Author: Jason Peng <jason@ufactory.cc>
 -->
-  <xacro:macro name="xarm_gripper_urdf" params="prefix:='' attach_to:='' rpy:='0 0 0' xyz:='0 0 0' ">
+  <xacro:macro name="xarm_gripper_urdf" params="prefix:='' attach_to:='' rpy:='0 0 0' xyz:='0 0 0' loop_joints:='false' ">
   <xacro:unless value="${attach_to == ''}">
     <joint name="${prefix}gripper_fix" type="fixed">
@@ -238,25 +238,27 @@
     <mimic joint="${prefix}drive_joint" multiplier="1" offset="0" />
   </joint>
-  <gazebo>
-    <joint name="${prefix}left_loop_joint" type="revolute">
-      <parent>${prefix}left_inner_knuckle</parent>
-      <child>${prefix}left_finger</child>
-      <pose>0 -0.015 0.015 0 0 0</pose>
-      <axis>
-        <xyz>1 0 0</xyz>
-        <use_parent_model_frame>true</use_parent_model_frame>
-      </axis>
-      <physics>
-        <ode>
-          <implicit_spring_damper>1</implicit_spring_damper>
-          <cfm_damping>0</cfm_damping>
-          <limit>
-            <cfm>1e-7</cfm>
-            <erp>0.8</erp>
-          </limit>
-        </ode>
-      </physics>
-    </joint>
-  </gazebo>
+  <xacro:if value="${loop_joints}">
+    <gazebo>
+      <joint name="${prefix}left_loop_joint" type="revolute">
+        <parent>${prefix}left_inner_knuckle</parent>
+        <child>${prefix}left_finger</child>
+        <pose>0 -0.015 0.015 0 0 0</pose>
+        <axis>
+          <xyz>1 0 0</xyz>
+          <use_parent_model_frame>true</use_parent_model_frame>
+        </axis>
+        <physics>
+          <ode>
+            <implicit_spring_damper>1</implicit_spring_damper>
+            <cfm_damping>0</cfm_damping>
+            <limit>
+              <cfm>1e-7</cfm>
+              <erp>0.8</erp>
+            </limit>
+          </ode>
+        </physics>
+      </joint>
+    </gazebo>
+  </xacro:if>
   <link
     name="${prefix}right_outer_knuckle">
@@ -444,25 +446,27 @@
     <mimic joint="${prefix}drive_joint" multiplier="1" offset="0" />
   </joint>
-  <gazebo>
-    <joint name="${prefix}right_loop_joint" type="revolute">
-      <parent>${prefix}right_inner_knuckle</parent>
-      <child>${prefix}right_finger</child>
-      <pose>0 0.015 0.015 0 0 0</pose>
-      <axis>
-        <xyz>1 0 0</xyz>
-        <use_parent_model_frame>true</use_parent_model_frame>
-      </axis>
-      <physics>
-        <ode>
-          <implicit_spring_damper>1</implicit_spring_damper>
-          <cfm_damping>0</cfm_damping>
-          <limit>
-            <cfm>1e-7</cfm>
-            <erp>0.8</erp>
-          </limit>
-        </ode>
-      </physics>
-    </joint>
-  </gazebo>
+  <xacro:if value="${loop_joints}">
+    <gazebo>
+      <joint name="${prefix}right_loop_joint" type="revolute">
+        <parent>${prefix}right_inner_knuckle</parent>
+        <child>${prefix}right_finger</child>
+        <pose>0 0.015 0.015 0 0 0</pose>
+        <axis>
+          <xyz>1 0 0</xyz>
+          <use_parent_model_frame>true</use_parent_model_frame>
+        </axis>
+        <physics>
+          <ode>
+            <implicit_spring_damper>1</implicit_spring_damper>
+            <cfm_damping>0</cfm_damping>
+            <limit>
+              <cfm>1e-7</cfm>
+              <erp>0.8</erp>
+            </limit>
+          </ode>
+        </physics>
+      </joint>
+    </gazebo>
+  </xacro:if>
   <link name="${prefix}link_tcp" />
   <joint

File: xarm_gripper/urdf/xarm_gripper_model.xacro (robot description, xacro)
@@ -8,8 +8,8 @@
   <xacro:include filename="$(find xarm_gripper)/urdf/xarm_gripper.transmission.xacro" />
   <xacro:include filename="$(find xarm_gripper)/urdf/xarm_gripper.gazebo.xacro" />
-  <xacro:macro name="load_gripper" params="prefix:='' attach_to:='' ns:='xarm' xyz:='0 0 0' rpy:='0 0 0' effort_control:='false' velocity_control:='false' robot_dof:=7 palm_link:=''">
+  <xacro:macro name="load_gripper" params="prefix:='' attach_to:='' ns:='xarm' xyz:='0 0 0' rpy:='0 0 0' effort_control:='false' velocity_control:='false' robot_dof:=7 palm_link:='' loop_joints:='true'">
     <!-- gazebo plugin -->
     <!-- <xacro:gazebo_ros_control_plugin namespace="${ns}"/> -->
-    <xacro:xarm_gripper_urdf prefix="${prefix}" attach_to="${attach_to}" xyz="${xyz}" rpy="${rpy}" />
+    <xacro:xarm_gripper_urdf prefix="${prefix}" attach_to="${attach_to}" xyz="${xyz}" rpy="${rpy}" loop_joints="${loop_joints}" />
     <xacro:xarm_gripper_transmission prefix="${prefix}" hard_interface="$(eval 'EffortJointInterface' if ${effort_control} else 'VelocityJointInterface' if ${velocity_control} else 'PositionJointInterface')" />
     <xacro:xarm_gripper_gazebo prefix="${prefix}" />
@@ -21,19 +21,23 @@
     </xacro:unless>
     <!-- mimic_joint_plugin has to be installed: -->
-<!--     <xacro:mimic_joint_plugin_gazebo name_prefix="${prefix}left_finger_joint"
-      following_joint="${prefix}drive_joint" mimic_joint="${prefix}left_finger_joint"
-      has_pid="true" multiplier="1.0" max_effort="10.0" /> -->
-<!--     <xacro:mimic_joint_plugin_gazebo name_prefix="${prefix}left_inner_knuckle_joint"
-      following_joint="${prefix}drive_joint" mimic_joint="${prefix}left_inner_knuckle_joint"
-      has_pid="true" multiplier="1.0" max_effort="10.0" /> -->
+    <!-- Only one mimic joint plug-in is needed when configuring parallel links with loop joints -->
     <xacro:mimic_joint_plugin_gazebo name_prefix="${prefix}right_outer_knuckle_joint"
       following_joint="${prefix}drive_joint" mimic_joint="${prefix}right_outer_knuckle_joint"
       has_pid="true" multiplier="1.0" max_effort="10.0" />
-<!--     <xacro:mimic_joint_plugin_gazebo name_prefix="${prefix}right_finger_joint"
-      following_joint="${prefix}drive_joint" mimic_joint="${prefix}right_finger_joint"
-      has_pid="true" multiplier="1.0" max_effort="10.0" /> -->
-<!--     <xacro:mimic_joint_plugin_gazebo name_prefix="${prefix}right_inner_knuckle_joint"
-      following_joint="${prefix}drive_joint" mimic_joint="${prefix}right_inner_knuckle_joint"
-      has_pid="true" multiplier="1.0" max_effort="10.0" /> -->
+    <!-- When configuring parallel links with mimic joint plug-ins, all passive joints must use mimic joint plug-ins -->
+    <xacro:unless value="${loop_joints}">
+      <xacro:mimic_joint_plugin_gazebo name_prefix="${prefix}left_finger_joint"
+        following_joint="${prefix}drive_joint" mimic_joint="${prefix}left_finger_joint"
+        has_pid="true" multiplier="1.0" max_effort="10.0" />
+      <xacro:mimic_joint_plugin_gazebo name_prefix="${prefix}left_inner_knuckle_joint"
+        following_joint="${prefix}drive_joint" mimic_joint="${prefix}left_inner_knuckle_joint"
+        has_pid="true" multiplier="1.0" max_effort="10.0" />
+      <xacro:mimic_joint_plugin_gazebo name_prefix="${prefix}right_finger_joint"
+        following_joint="${prefix}drive_joint" mimic_joint="${prefix}right_finger_joint"
+        has_pid="true" multiplier="1.0" max_effort="10.0" />
+      <xacro:mimic_joint_plugin_gazebo name_prefix="${prefix}right_inner_knuckle_joint"
+        following_joint="${prefix}drive_joint" mimic_joint="${prefix}right_inner_knuckle_joint"
+        has_pid="true" multiplier="1.0" max_effort="10.0" />
+    </xacro:unless>
   </xacro:macro>
 </robot>

Commit message: Update gripper collision

File: xarm_gripper/urdf/xarm_gripper.urdf.xacro (robot description, xacro)
@@ -142,8 +142,16 @@
     <collision>
       <origin
-        xyz="0 -0.019 0.04"
-        rpy="0 0 0" />
-      <geometry>
-        <box size="0.032 0.014 0.042"/>
+        xyz="0 -0.0224 0.04"
+        rpy="0 0 0" />
+      <geometry>
+        <box size="0.032 0.0072 0.042"/>
+      </geometry>
+    </collision>
+    <collision>
+      <origin
+        xyz="0 -0.0154 0.036"
+        rpy="0 0 0" />
+      <geometry>
+        <box size="0.032 0.0068 0.034"/>
       </geometry>
     </collision>
@@ -350,8 +358,16 @@
     <collision>
       <origin
-        xyz="0 0.019 0.04"
-        rpy="0 0 0" />
-      <geometry>
-        <box size="0.032 0.014 0.042"/>
+        xyz="0 0.0224 0.04"
+        rpy="0 0 0" />
+      <geometry>
+        <box size="0.032 0.0072 0.042"/>
+      </geometry>
+    </collision>
+    <collision>
+      <origin
+        xyz="0 0.0154 0.036"
+        rpy="0 0 0" />
+      <geometry>
+        <box size="0.032 0.0068 0.034"/>
       </geometry>
     </collision>

Commit message: disable unecessary damping

File: xarm_gripper/urdf/xarm_gripper.urdf.xacro (robot description, xacro)
@@ -106,5 +106,5 @@
       lower="0"
       upper="0.85"
-      effort="50"
+      effort="1.0"
       velocity="2" />
     <dynamics
@@ -182,7 +182,7 @@
       effort="50"
       velocity="2" />
-    <dynamics
-      damping="1.0"
-      friction="0" />
+    <!--<dynamics-->
+    <!--  damping="1.0"-->
+    <!--  friction="0" />-->
     <mimic joint="${prefix}drive_joint" multiplier="1" offset="0" />
   </joint>
@@ -241,7 +241,7 @@
       effort="50"
       velocity="2" />
-    <dynamics
-      damping="1.0"
-      friction="0" />
+    <!--<dynamics-->
+    <!--  damping="1.0"-->
+    <!--  friction="0" />-->
     <mimic joint="${prefix}drive_joint" multiplier="1" offset="0" />
   </joint>
@@ -256,14 +256,14 @@
           <use_parent_model_frame>false</use_parent_model_frame>
         </axis>
-        <physics>
-          <ode>
-            <implicit_spring_damper>1</implicit_spring_damper>
-            <cfm_damping>0</cfm_damping>
-            <limit>
-              <cfm>1e-7</cfm>
-              <erp>0.8</erp>
-            </limit>
-          </ode>
-        </physics>
+        <!--<physics>-->
+        <!--  <ode>-->
+        <!--    <implicit_spring_damper>1</implicit_spring_damper>-->
+        <!--    <cfm_damping>0</cfm_damping>-->
+        <!--    <limit>-->
+        <!--      <cfm>1e-7</cfm>-->
+        <!--      <erp>0.8</erp>-->
+        <!--    </limit>-->
+        <!--  </ode>-->
+        <!--</physics>-->
       </joint>
     </gazebo>
@@ -323,7 +323,7 @@
       effort="50"
       velocity="2" />
-    <dynamics
-      damping="1.0"
-      friction="0" />
+    <!--<dynamics-->
+    <!--  damping="1.0"-->
+    <!--  friction="0" />-->
     <mimic joint="${prefix}drive_joint" multiplier="1" offset="0" />
   </joint>
@@ -398,7 +398,7 @@
       effort="50"
       velocity="2" />
-    <dynamics
-      damping="1.0"
-      friction="0" />
+    <!--<dynamics-->
+    <!--  damping="1.0"-->
+    <!--  friction="0" />-->
     <mimic joint="${prefix}drive_joint" multiplier="1" offset="0" />
   </joint>
@@ -455,9 +455,9 @@
       lower="0"
       upper="0.85"
-      effort="50"
+      effort="0.5"
       velocity="2" />
-    <dynamics
-      damping="1.0"
-      friction="0" />
+    <!--<dynamics-->
+    <!--  damping="1.0"-->
+    <!--  friction="0" />-->
     <mimic joint="${prefix}drive_joint" multiplier="1" offset="0" />
   </joint>
@@ -472,14 +472,14 @@
           <use_parent_model_frame>false</use_parent_model_frame>
         </axis>
-        <physics>
-          <ode>
-            <implicit_spring_damper>1</implicit_spring_damper>
-            <cfm_damping>0</cfm_damping>
-            <limit>
-              <cfm>1e-7</cfm>
-              <erp>0.8</erp>
-            </limit>
-          </ode>
-        </physics>
+        <!--<physics>-->
+        <!--  <ode>-->
+        <!--    <implicit_spring_damper>1</implicit_spring_damper>-->
+        <!--    <cfm_damping>0</cfm_damping>-->
+        <!--    <limit>-->
+        <!--      <cfm>1e-7</cfm>-->
+        <!--      <erp>0.8</erp>-->
+        <!--    </limit>-->
+        <!--  </ode>-->
+        <!--</physics>-->
       </joint>
     </gazebo>

Commit message: Update gripper

File: xarm_gripper/urdf/xarm_gripper.urdf.xacro (robot description, xacro)
@@ -47,8 +47,16 @@
     <collision>
       <origin
-        xyz="-0.0015 0 0.0515"
-        rpy="0 0 0" />
-      <geometry>
-        <box size="0.053 0.12 0.103"/>
+        xyz="-0.0015 0 0.055"
+        rpy="0 0 0" />
+      <geometry>
+        <box size="0.053 0.1 0.1"/>
+      </geometry>
+    </collision>
+    <collision>
+      <origin
+        xyz="0.03 -0.062 0.025"
+        rpy="0 0 0" />
+      <geometry>
+        <box size="0.076 0.024 0.04"/>
       </geometry>
     </collision>
