Commit message: Rename finger_extension to finger_tip

File: xarm_gripper/urdf/finger_tip.xacro (robot description, xacro)
@@ -1,5 +1,5 @@
 <?xml version="1.0" encoding="UTF-8"?>
 <robot xmlns:xacro="http://www.ros.org/wiki/xacro">
-  <xacro:macro name="finger_extension" params="name parent *origin collide_without_contact:='false'">
+  <xacro:macro name="finger_tip" params="name parent *origin collide_without_contact:='false'">
     <xacro:macro name="box_inertial" params="mass origin d w h">
       <inertial>
@@ -9,10 +9,10 @@
       </inertial>
     </xacro:macro>
-    <joint name="${name}_finger_extension_joint" type="fixed">
+    <joint name="${name}_finger_tip_joint" type="fixed">
       <xacro:insert_block name="origin"/>
       <parent link="${parent}"/>
-      <child link="${name}_finger_extension_link"/>
+      <child link="${name}_finger_tip_link"/>
     </joint>
-    <link name="${name}_finger_extension_link">
+    <link name="${name}_finger_tip_link">
       <visual>
         <origin xyz="0 0 0.004" rpy="0 0 0"/>
@@ -32,5 +32,5 @@
       <xacro:box_inertial mass="0.019" origin="0 0 0" d="0.040" w="0.032" h="0.007"/>
     </link>
-    <gazebo reference="${name}_finger_extension_link">
+    <gazebo reference="${name}_finger_tip_link">
       <kp>100000.0</kp>
       <kd>100.0</kd>

File: xarm_gripper/urdf/xarm_gripper.urdf.xacro (robot description, xacro)
@@ -4,5 +4,5 @@
   Author: Jason Peng <jason@ufactory.cc>
 -->
-  <xacro:macro name="xarm_gripper_urdf" params="prefix:='' attach_to:='' rpy:='0 0 0' xyz:='0 0 0' loop_joints:='false' use_default_finger_extension:='true'">
+  <xacro:macro name="xarm_gripper_urdf" params="prefix:='' attach_to:='' rpy:='0 0 0' xyz:='0 0 0' loop_joints:='false' use_default_finger_tip:='true'">
   <xacro:unless value="${attach_to == ''}">
     <joint name="${prefix}gripper_fix" type="fixed">
@@ -481,12 +481,12 @@
       link="${prefix}link_tcp" />
   </joint>
-  <xacro:if value="${use_default_finger_extension}">
-    <xacro:include filename="$(find xarm_gripper)/urdf/finger_extension.xacro"/>
-    <xacro:finger_extension name="left" parent="${prefix}left_finger">
+  <xacro:if value="${use_default_finger_tip}">
+    <xacro:include filename="$(find xarm_gripper)/urdf/finger_tip.xacro"/>
+    <xacro:finger_tip name="left" parent="${prefix}left_finger">
       <origin rpy="0 0 0" xyz="0 -0.0225 0.037"/>
-    </xacro:finger_extension>
-    <xacro:finger_extension name="right" parent="${prefix}right_finger">
+    </xacro:finger_tip>
+    <xacro:finger_tip name="right" parent="${prefix}right_finger">
       <origin rpy="0 0 0" xyz="0 0.0225 0.037"/>
-    </xacro:finger_extension>
+    </xacro:finger_tip>
   </xacro:if>
   </xacro:macro>

File: xarm_gripper/urdf/xarm_gripper_model.xacro (robot description, xacro)
@@ -8,8 +8,8 @@
   <xacro:include filename="$(find xarm_gripper)/urdf/xarm_gripper.transmission.xacro" />
   <xacro:include filename="$(find xarm_gripper)/urdf/xarm_gripper.gazebo.xacro" />
-  <xacro:macro name="load_gripper" params="prefix:='' attach_to:='' ns:='xarm' xyz:='0 0 0' rpy:='0 0 0' effort_control:='false' velocity_control:='false' robot_dof:=7 palm_link:='' loop_joints:='true' collide_without_contact:='false' use_default_finger_extension:='true'">
+  <xacro:macro name="load_gripper" params="prefix:='' attach_to:='' ns:='xarm' xyz:='0 0 0' rpy:='0 0 0' effort_control:='false' velocity_control:='false' robot_dof:=7 palm_link:='' loop_joints:='true' collide_without_contact:='false' use_default_finger_tip:='true'">
     <!-- gazebo plugin -->
     <!-- <xacro:gazebo_ros_control_plugin namespace="${ns}"/> -->
-    <xacro:xarm_gripper_urdf prefix="${prefix}" attach_to="${attach_to}" xyz="${xyz}" rpy="${rpy}" loop_joints="${loop_joints}" use_default_finger_extension="${use_default_finger_extension}"/>
+    <xacro:xarm_gripper_urdf prefix="${prefix}" attach_to="${attach_to}" xyz="${xyz}" rpy="${rpy}" loop_joints="${loop_joints}" use_default_finger_tip="${use_default_finger_tip}"/>
     <xacro:xarm_gripper_transmission prefix="${prefix}" hard_interface="$(eval 'EffortJointInterface' if ${effort_control} else 'VelocityJointInterface' if ${velocity_control} else 'PositionJointInterface')" />
     <xacro:xarm_gripper_gazebo prefix="${prefix}" collide_without_contact="${collide_without_contact}" />
